File: docs/schematics/eagle/door-strike-schematic.sch (EAGLE design)
At the start: 9 parts, among them IC1 LD1117, T1 TIP120

Commit message: more schematic organization
Connections:
- new net N$3: U$2.GND@3
- new net N$4: C2.2
- net GND: no longer C2.2, U$2.GND@3
Other:
- moved on the sheet: R1, T1
Changed lines of the file:
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@@
 </plain>
 <instances>
-<instance part="T1" gate="1" x="48.26" y="53.34"/>
-<instance part="R1" gate="G$1" x="35.56" y="53.34"/>
+<instance part="T1" gate="1" x="48.26" y="45.72"/>
+<instance part="R1" gate="G$1" x="35.56" y="45.72"/>
 <instance part="D1" gate="1" x="58.42" y="73.66"/>
 <instance part="JST1" gate="G$1" x="63.5" y="91.44" rot="R90"/>
 <instance part="GND1" gate="1" x="50.8" y="25.4"/>
-<instance part="GND2" gate="1" x="40.64" y="25.4"/>
+<instance part="GND2" gate="1" x="40.64" y="50.8"/>
 <instance part="12VDC" gate="G$1" x="73.66" y="58.42"/>
 <instance part="IC1" gate="G$1" x="55.88" y="104.14" rot="R180"/>
@@
 <instance part="C2" gate="G$1" x="88.9" y="88.9"/>
 <instance part="GND5" gate="1" x="88.9" y="25.4"/>
-<instance part="U$2" gate="G$1" x="5.08" y="53.34" rot="R180"/>
+<instance part="U$2" gate="G$1" x="5.08" y="45.72" rot="R180"/>
 </instances>
 <busses>
@@
 <pinref part="T1" gate="1" pin="E"/>
 <pinref part="GND1" gate="1" pin="GND"/>
-<wire x1="50.8" y1="48.26" x2="50.8" y2="27.94" width="0.1524" layer="91"/>
+<wire x1="50.8" y1="40.64" x2="50.8" y2="27.94" width="0.1524" layer="91"/>
 </segment>
 <segment>
@@
 </segment>
 <segment>
-<pinref part="U$2" gate="G$1" pin="GND@3"/>
-<wire x1="25.4" y1="58.42" x2="40.64" y2="58.42" width="0.1524" layer="91"/>
 <pinref part="C1" gate="G$1" pin="-"/>
-<wire x1="40.64" y1="83.82" x2="40.64" y2="58.42" width="0.1524" layer="91"/>
+<wire x1="40.64" y1="83.82" x2="40.64" y2="53.34" width="0.1524" layer="91"/>
 <pinref part="GND2" gate="1" pin="GND"/>
-<wire x1="40.64" y1="58.42" x2="40.64" y2="27.94" width="0.1524" layer="91"/>
-<junction x="40.64" y="58.42"/>
-</segment>
-<segment>
-<pinref part="C2" gate="G$1" pin="2"/>
-<wire x1="88.9" y1="83.82" x2="88.9" y2="25.4" width="0.1524" layer="91"/>
 </segment>
 </net>
@@
 <net name="N$7" class="0">
 <segment>
-<wire x1="-22.86" y1="104.14" x2="-22.86" y2="55.88" width="0.1524" layer="91"/>
+<wire x1="-22.86" y1="104.14" x2="-22.86" y2="48.26" width="0.1524" layer="91"/>
 <pinref part="U$2" gate="G$1" pin="+3.3V"/>
-<wire x1="-22.86" y1="55.88" x2="-15.24" y2="55.88" width="0.1524" layer="91"/>
+<wire x1="-22.86" y1="48.26" x2="-15.24" y2="48.26" width="0.1524" layer="91"/>
 <pinref part="IC1" gate="G$1" pin="VOUT"/>
 <wire x1="45.72" y1="104.14" x2="40.64" y2="104.14" width="0.1524" layer="91"/>
@@
 <wire x1="50.8" y1="91.44" x2="50.8" y2="73.66" width="0.1524" layer="91"/>
 <pinref part="D1" gate="1" pin="A"/>
-<wire x1="50.8" y1="73.66" x2="50.8" y2="58.42" width="0.1524" layer="91"/>
+<wire x1="50.8" y1="73.66" x2="50.8" y2="50.8" width="0.1524" layer="91"/>
 <wire x1="50.8" y1="73.66" x2="55.88" y2="73.66" width="0.1524" layer="91"/>
 <junction x="50.8" y="73.66"/>
@@
 <pinref part="R1" gate="G$1" pin="1"/>
 <pinref part="U$2" gate="G$1" pin="P0.05/AIN6"/>
-<wire x1="30.48" y1="53.34" x2="25.4" y2="53.34" width="0.1524" layer="91"/>
+<wire x1="30.48" y1="45.72" x2="25.4" y2="45.72" width="0.1524" layer="91"/>
 </segment>
 </net>
@@
 <segment>
 <pinref part="R1" gate="G$1" pin="2"/>
-<wire x1="40.64" y1="53.34" x2="48.26" y2="53.34" width="0.1524" layer="91"/>
+<wire x1="40.64" y1="45.72" x2="48.26" y2="45.72" width="0.1524" layer="91"/>
 </segment>
 </net>
+<net name="N$4" class="0">
+<segment>
+<pinref part="C2" gate="G$1" pin="2"/>
+<wire x1="88.9" y1="83.82" x2="88.9" y2="25.4" width="0.1524" layer="91"/>
+</segment>
+</net>
+<net name="N$3" class="0">
+<segment>
+<pinref part="U$2" gate="G$1" pin="GND@3"/>
+<wire x1="25.4" y1="50.8" x2="40.64" y2="50.8" width="0.1524" layer="91"/>
+</segment>
+</net>
